File: inv24to120V.kicad_pcb (KiCad board)
At the start: 2 copper layers, 105 x 155 mm, 130 parts, among them IC1 FSAM50SM60A, J1 Conn_02x13_Odd_Even, J5 Screw_Terminal_01x02, J6 Screw_Terminal_01x03, J7 Screw_Terminal_01x03, J8 Screw_Terminal_01x03, J9 Screw_Terminal_01x02, K1 J0971CS5VDC.45, Q1 IRFZ44NPBF, Q2 IRFZ44NPBF, Q3 2SC1815, Q4 2SC1815, Q5 2SA1015, Q6 2SA1015, Q7 2SC1815, U10 PC817, U2 LM2576HVT-5, U3 ACS712ELCTR30AT, U4 ACS712ELCTR30AT, U5 LM2576HVT-5, U6 ISO7340CDW, U7 ISO7340CDW, U8 AMC1300BDWVR, U9 PC817

Commit message: route done
Parts:
- removed F2: 3544-2, inv24VLib:FUSE_3544-2
- added C39: 104, Capacitor_SMD:C_0805_2012Metric, F.Cu at (61.0, 85.9)
- added C40: 100uF/50V, Capacitor_THT:CP_Radial_D8.0mm_P5.00mm, F.Cu at (116.3, 108.7)
- added C41: 104, Capacitor_SMD:C_0805_2012Metric, F.Cu at (53.2, 116.8)
- added C42: 104, Capacitor_SMD:C_0805_2012Metric, F.Cu at (56.5, 116.8)
- added C43: 22uF/10V, Capacitor_SMD:C_1210_3225Metric_Pad1.33x2.70mm_HandSolder, F.Cu at (63.5, 110.1)
- added C44: 22uF/10V, Capacitor_SMD:C_1210_3225Metric_Pad1.33x2.70mm_HandSolder, F.Cu at (108.1, 100.9)
- added U11: LM1117MP-3.3, Package_TO_SOT_SMD:SOT-223-3_TabPin2, F.Cu at (55.7, 109.8)
- C35: value 47uF/50V -> 22uF/10V; footprint Capacitor_THT:CP_Radial_D8.0mm_P5.00mm -> Capacitor_SMD:C_1210_3225Metric_Pad1.33x2.70mm_HandSolder
- D1, D2, D6: footprint Diode_THT:D_DO-201AD_P15.24mm_Horizontal -> Diode_THT:D_DO-201AD_P3.81mm_Vertical_AnodeUp
- D7: footprint Diode_THT:D_DO-41_SOD81_P10.16mm_Horizontal -> Diode_THT:D_DO-201AD_P3.81mm_Vertical_AnodeUp
- Q3, Q4: value 2SC1815 -> 2SC1815_SOT32; footprint Package_TO_SOT_THT:TO-92_Inline -> Package_TO_SOT_SMD:SOT-23-3
- Q5, Q6: value 2SA1015 -> 2SA1015_SOT32; footprint Package_TO_SOT_THT:TO-92_Inline -> Package_TO_SOT_SMD:SOT-23-3
- Q7: footprint Package_TO_SOT_THT:TO-92_Inline -> Package_TO_SOT_SMD:SOT-23-3
- R1, R2, R3, R4, R42, R45, R46, R48, R5, R6: footprint Resistor_THT:R_Axial_DIN0207_L6.3mm_D2.5mm_P10.16mm_Horizontal -> Resistor_SMD:R_0805_2012Metric_Pad1.20x1.40mm_HandSolder
- R11, R12, R13: footprint Resistor_THT:R_Axial_DIN0309_L9.0mm_D3.2mm_P15.24mm_Horizontal -> Resistor_THT:R_Axial_DIN0309_L9.0mm_D3.2mm_P20.32mm_Horizontal
- R47: value 470 -> 2k; footprint Resistor_THT:R_Axial_DIN0207_L6.3mm_D2.5mm_P10.16mm_Horizontal -> Resistor_SMD:R_0805_2012Metric_Pad1.20x1.40mm_HandSolder
- moved C38 74.4 mm to (128.8, 92.9), turned to 90 degrees
- moved R48 68.2 mm to (87.5, 108.0), turned to -90 degrees
- moved R44 49.7 mm to (111.7, 96.0)
- moved R5 48.4 mm to (95.0, 108.0), turned to -90 degrees
- moved H1 46.1 mm to (153.0, 105.0)
- moved R6 45.5 mm to (92.5, 108.0), turned to -90 degrees
- moved R10 37.7 mm to (76.5, 60.0)
- moved R8 37.0 mm to (72.6, 60.0)
- moved L4 36.5 mm to (124.0, 163.5), turned to 180 degrees
- moved R9 34.1 mm to (76.5, 65.0)
- moved C22 33.2 mm to (134.0, 128.0), turned to -90 degrees
- moved R7 32.5 mm to (72.5, 65.0)
- moved C37 32.4 mm to (90.0, 108.0), turned to 90 degrees
- moved D8 31.5 mm to (151.5, 142.5)
- moved R2 27.4 mm to (62.5, 151.0), turned to 180 degrees
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Connections:
- BX1 pad 2: +3.3V -> +5V
- J1 pad 10: +3.3V -> unconnected-(J1-Pin_10-Pad10)
- J1 pad 9: +3.3V -> unconnected-(J1-Pin_9-Pad9)
- J5 pad 2: Net-(J5-Pin_2) -> GND
- J9 pad 2: Net-(J9-Pin_2) -> GND
- Q3 pad 1: GND -> Net-(Q3-B)
- Q3 pad 2: Net-(Q3-C) -> GND
- Q3 pad 3: Net-(Q3-B) -> Net-(Q3-C)
- Q4 pad 1: GND -> Net-(Q4-B)
- Q4 pad 2: Net-(Q4-C) -> GND
- Q4 pad 3: Net-(Q4-B) -> Net-(Q4-C)
- Q5 pad 1: +5V -> Net-(Q3-B)
- Q5 pad 2: Net-(Q3-C) -> +5V
- Q5 pad 3: Net-(Q3-B) -> Net-(Q3-C)
- Q6 pad 1: +5V -> Net-(Q4-B)
- Q6 pad 2: Net-(Q4-C) -> +5V
- Q6 pad 3: Net-(Q4-B) -> Net-(Q4-C)
- Q7 pad 1: GND -> Net-(Q7-B)
- Q7 pad 2: Net-(D7-A) -> GND
- Q7 pad 3: Net-(Q7-B) -> Net-(D7-A)
- R47 pad 1: Net-(J9-Pin_2) -> +24V
- R47 pad 2: GND -> Net-(R47-Pad2)
- U9 pad 1: +5V -> Net-(R47-Pad2)
Routing:
- net GND2: track 145.6 -> 390.9 mm, vias 7 -> 13
- net GND: track 288.0 -> 518.6 mm, vias 0 -> 21
- net +5VP: track 89.6 -> 291.0 mm, vias 8 -> 10
- net +5V: track 106.5 -> 295.9 mm, vias 0 -> 9
- net +15V: track 105.6 -> 261.9 mm, vias 1 -> 2
- net GNDPWR: track 124.2 -> 279.8 mm, vias 0 -> 6
- net VTH_IPM: track 0.00 -> 135.6 mm, vias 0 -> 1
- net Net-(IC1-RTH): track 0.00 -> 131.5 mm, vias 0 -> 1
- net DIGITAL_CMD: track 5.33 -> 94.6 mm
- net Earth_Protective: track 0.00 -> 87.7 mm
- net U_sensor: track 0.00 -> 76.3 mm, vias 0 -> 2
- net Net-(Q4-B): track 0.00 -> 75.2 mm, vias 0 -> 2
- net Net-(Q3-B): track 0.00 -> 71.1 mm, vias 0 -> 4
- net RELAY_TRIP: track 0.00 -> 56.7 mm, vias 0 -> 4
- net FAULT_IPM: track 0.00 -> 50.1 mm, vias 0 -> 2
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Other:
- outline, holes or cut-outs redrawn

Commit message: edit reference
Routing:
- net U_sensor: track 76.3 -> 76.2 mm, vias 2 -> 18

Commit message: rout finish
Parts:
- moved L2 14.5 mm to (152.0, 174.3), turned to 180 degrees
- moved C4 12.4 mm to (145.2, 163.7), turned to 90 degrees
- moved C40 11.5 mm to (107.7, 116.3), turned to 0 degrees
- moved C3 11.0 mm to (138.0, 158.8), turned to 90 degrees
- moved D1 10.5 mm to (65.0, 118.0), turned to 90 degrees
- moved C43 10.4 mm to (53.5, 107.1), turned to -90 degrees
- moved U2 9.00 mm to (53.5, 119.9)
- moved Q1 8.50 mm to (53.5, 131.1)
- moved L3 8.31 mm to (141.2, 168.5), turned to 180 degrees
- moved D2 6.24 mm to (144.7, 154.0), turned to 0 degrees
- moved C41 5.66 mm to (58.8, 115.5)
- moved L1 5.53 mm to (67.5, 124.0), turned to -90 degrees
- moved C38 5.08 mm to (128.5, 87.9), turned to 45 degrees
- moved C35 4.89 mm to (109.8, 108.1)
- moved C42 4.70 mm to (61.0, 115.5)
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Routing:
- net GND: track 518.6 -> 551.3 mm, vias 21 -> 22
- net +15V: track 261.9 -> 240.0 mm, vias 2 -> 3
- net ANALOG_CMD: track 47.3 -> 32.5 mm, vias 2 -> 1
- net Net-(D2-K): track 16.2 -> 27.6 mm
- net +5V: track 295.9 -> 285.8 mm, vias 9 -> 10
- net GND2: track 390.9 -> 381.9 mm, vias 13 -> 11
- net VTH_IPM: track 135.6 -> 144.3 mm
- net +3.3V: track 139.0 -> 146.9 mm
- net Net-(Q1-G): track 14.7 -> 22.3 mm
- net +5VP: track 291.0 -> 283.5 mm
- net H+15V: track 33.4 -> 39.9 mm
- net +24V: track 121.8 -> 116.9 mm
- net Net-(J6-Pin_3): track 20.3 -> 25.0 mm, vias 1 -> 0
- net Net-(BX5-Pad2): track 5.84 -> 10.2 mm
- net FAULT_IPM: track 50.1 -> 53.7 mm
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