File: inv24to120V.kicad_pcb (KiCad board)
At the start: 2 copper layers, 105 x 155 mm, 133 parts, among them IC1 FSAM50SM60A, J1 Conn_02x13_Odd_Even_MountingP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, J10 Screw_Terminal_01x01, J11 Screw_Terminal_01x01, J12 Screw_Terminal_01x01, J2 Conn_02x13_Odd_Even_MountingP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, J3 Screw_Terminal_01x01, J4 Conn_02x05_Odd_Even_MountingP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, J5 Screw_Terminal_01x02, J6 Screw_Terminal_01x03, J7 Screw_Terminal_01x03, J8 Screw_Terminal_01x03, J9 Screw_Terminal_01x02, K1 J0971CS5VDC.45, Q1 IRFZ44NPBF, Q2 IRFZ44NPBF, Q3 2SC1815, Q4 2SC1815, Q5 2SA1015, Q6 2SA1015, Q7 2SC1815, U1 ESP32-DEVKITC-32D, U10 PC817, U2 LM2576HVT-5, U3 ACS712ELCTR30AT, U4 ACS712ELCTR30AT, U5 LM2576HVT-5, U6 ISO7340CDW, U7 ISO7340CDW, U8 AMC1300BDWVR, U9 PC817

Commit message: to pcb fix error
Parts:
- removed BX1, BX2, BX3, BX4, BX5, BX6: 0, Resistor_THT:R_Axial_DIN0207_L6.3mm_D2.5mm_P10.16mm_Horizontal
- removed C1, C2, C4: 100uF/50V, Capacitor_THT:CP_Radial_D8.0mm_P5.00mm
- removed C10, C11, C16, C17, C18, C20, C21, C23, C26, C32, C33, C34, C36, C37, C6, C7, C9: 104, Capacitor_SMD:C_0805_2012Metric
- removed C12, C25, C27, C28, C29, C30, C31, C5, C8: 102, Capacitor_SMD:C_0805_2012Metric
- removed C13, C14, C15: 22uF/25V, Capacitor_SMD:C_0805_2012Metric
- removed C22: 470uF/400V, inv24VLib:CAPPRD1000W160D3600H5200
- removed C24: 333, Capacitor_SMD:C_0805_2012Metric
- removed C3: 470uF/50V, Capacitor_THT:CP_Radial_D8.0mm_P5.00mm
- removed C35: 47uF/50V, Capacitor_THT:CP_Radial_D8.0mm_P5.00mm
- removed D1, D2, D6: 1N5822, Diode_THT:D_DO-201AD_P15.24mm_Horizontal
- removed D3, D4, D5: 1N4937, Diode_THT:D_DO-35_SOD27_P10.16mm_Horizontal
- removed D7: 1N4002, Diode_THT:D_DO-41_SOD81_P10.16mm_Horizontal
- removed D8, D9: BYV29X-500, inv24VLib:TO507P1020X460X2000-2
- removed F1, F2: 3544-2, inv24VLib:FUSE_3544-2
- removed IC1: FSAM50SM60A, inv24VLib:DIP-32
- removed J1, J2: Conn_02x13_Odd_Even_MountingPin, Connector_IDC:IDC-Header_2x13_P2.54mm_Vertical
- removed J10, J11, J12, J3: Screw_Terminal_01x01, TerminalBlock_Wuerth:Wuerth_REDCUBE-THR_WP-THRBU_74650073_THR
- removed J4: Conn_02x05_Odd_Even_MountingPin, Connector_IDC:IDC-Header_2x05_P2.54mm_Vertical
- removed J5: Screw_Terminal_01x02, TerminalBlock_Dinkle:TerminalBlock_Dinkle_DT-55-B01X-02_P10.00mm
- removed J6: Screw_Terminal_01x03, TerminalBlock_Phoenix:TerminalBlock_Phoenix_MKDS-1,5-3-5.08_1x03_P5.08mm_Horizontal
- removed J7: Screw_Terminal_01x03, TerminalBlock_Dinkle:TerminalBlock_Dinkle_DT-55-B01X-03_P10.00mm
- removed J8: Screw_Terminal_01x03, TerminalBlock_Phoenix:TerminalBlock_Phoenix_MKDS-1,5-3_1x03_P5.00mm_Horizontal
- removed J9: Screw_Terminal_01x02, TerminalBlock_Phoenix:TerminalBlock_Phoenix_MKDS-1,5-2-5.08_1x02_P5.08mm_Horizontal
- removed K1: J0971CS5VDC.45, inv24VLib:RELAY_J0971CS5VDC.45
- removed L1, L2, L3: 100uH, Inductor_THT:L_Radial_D10.0mm_P5.00mm_Neosid_SD12k_style3
- removed L4: 22uH, inv24VLib:IND_HCTI-10-20.0
- removed Q1, Q2: IRFZ44NPBF, Package_TO_SOT_THT:TO-220-3_Vertical
- removed Q3, Q4, Q7: 2SC1815, Package_TO_SOT_THT:TO-92_Inline
- removed Q5, Q6: 2SA1015, Package_TO_SOT_THT:TO-92_Inline
- removed R1, R2: 10, Resistor_THT:R_Axial_DIN0207_L6.3mm_D2.5mm_P10.16mm_Horizontal
- removed R10, R20, R21, R7, R8, R9: 2K, Resistor_SMD:R_0805_2012Metric
- removed R11, R12, R13: 5.6, Resistor_THT:R_Axial_DIN0207_L6.3mm_D2.5mm_P10.16mm_Horizontal
- removed R14, R15, R16: 20, Resistor_THT:R_Axial_DIN0207_L6.3mm_D2.5mm_P10.16mm_Horizontal
- removed R17, R18: 1M/2W, Resistor_THT:R_Axial_DIN0414_L11.9mm_D4.5mm_P15.24mm_Horizontal
- removed R19: 1K, Resistor_THT:R_Axial_DIN0207_L6.3mm_D2.5mm_P10.16mm_Horizontal
- removed R22: 470, Resistor_SMD:R_0805_2012Metric
- removed R23: 390, Resistor_SMD:R_0805_2012Metric
- removed R24: 3.9K, Resistor_SMD:R_0805_2012Metric
- removed R25: 45, Resistor_SMD:R_0805_2012Metric
- removed R26, R27, R28, R35, R36, R37: 4.7K, Resistor_SMD:R_0805_2012Metric
- removed R29, R30, R31, R32, R33, R34: 100, Resistor_SMD:R_0805_2012Metric
- removed R3, R4, R40: 10K, Resistor_THT:R_Axial_DIN0207_L6.3mm_D2.5mm_P10.16mm_Horizontal
- removed R42, R44, R46, R48: 4.7K, Resistor_THT:R_Axial_DIN0207_L6.3mm_D2.5mm_P10.16mm_Horizontal
- removed R45, R47: 470, Resistor_THT:R_Axial_DIN0207_L6.3mm_D2.5mm_P10.16mm_Horizontal
- removed R5, R6: 100, Resistor_THT:R_Axial_DIN0207_L6.3mm_D2.5mm_P10.16mm_Horizontal
- removed U1: ESP32-DEVKITC-32D, inv24VLib:MODULE_ESP32-DEVKITC-32D
- removed U10, U9: PC817, Package_DIP:DIP-4_W7.62mm
- removed U2, U5: LM2576HVT-5, Package_TO_SOT_THT:TO-220-5_Vertical
- removed U3, U4: ACS712ELCTR30AT, inv24VLib:SOIC127P600X175-8N
- removed U6, U7: ISO7340CDW, inv24VLib:SOIC127P1030X265-16N
- removed U8: AMC1300BDWVR, inv24VLib:SOIC127P1150X280-8N
- removed X1: ~, inv24VLib:ee42208x8p
Other:
- board size 105 x 155 mm -> 220 x 150 mm

Commit message: start place parts
Parts:
- added BC1: 104, Capacitor_SMD:C_0805_2012Metric_Pad1.18x1.45mm_HandSolder, F.Cu at (348.9, 116.0)
- added BC2: 104, Capacitor_SMD:C_0805_2012Metric_Pad1.18x1.45mm_HandSolder, F.Cu at (348.9, 119.0)
- added BX1: BLM31KN801SH1L, Resistor_SMD:R_1206_3216Metric_Pad1.30x1.75mm_HandSolder, F.Cu at (337.5, 174.9)
- added BX2: BLM31KN801SH1L, Resistor_SMD:R_1206_3216Metric_Pad1.30x1.75mm_HandSolder, F.Cu at (337.5, 178.2)
- added BX3: BLM31KN801SH1L, Resistor_SMD:R_1206_3216Metric_Pad1.30x1.75mm_HandSolder, F.Cu at (337.5, 181.5)
- added BX4: BLM31KN801SH1L, Resistor_SMD:R_1206_3216Metric_Pad1.30x1.75mm_HandSolder, F.Cu at (337.5, 184.8)
- added C1: 2200uF/50V, Capacitor_THT:CP_Radial_D12.5mm_P7.50mm, F.Cu at (64.5, 26.3)
- added C10: 104, Capacitor_SMD:C_0805_2012Metric, F.Cu at (340.7, 31.7)
- added C11: 104, Capacitor_SMD:C_0805_2012Metric, F.Cu at (340.7, 34.7)
- added C12: 102, Capacitor_SMD:C_0805_2012Metric, F.Cu at (345.2, 13.6)
- added C13: 22uF/25V, Capacitor_SMD:C_0805_2012Metric, F.Cu at (345.2, 16.6)
- added C14: 22uF/25V, Capacitor_SMD:C_0805_2012Metric, F.Cu at (345.2, 19.6)
- added C15: 22uF/25V, Capacitor_SMD:C_0805_2012Metric, F.Cu at (345.2, 22.6)
- added C16: 104, Capacitor_SMD:C_0805_2012Metric, F.Cu at (345.2, 25.6)
- added C17: 104, Capacitor_SMD:C_0805_2012Metric, F.Cu at (345.2, 28.6)
- added C18: 104, Capacitor_SMD:C_0805_2012Metric, F.Cu at (345.2, 31.7)
- added C19: 104, Capacitor_SMD:C_0805_2012Metric, F.Cu at (345.2, 34.7)
- added C2: 470uF/25V, Capacitor_SMD:CP_Elec_10x12.5, F.Cu at (179.4, 153.3)
- added C20: 104, Capacitor_SMD:C_0805_2012Metric, F.Cu at (349.6, 13.6)
- added C21: 104, Capacitor_SMD:C_0805_2012Metric, F.Cu at (349.6, 16.6)
- added C22: 470uF/400V, inv24VLib:CAPPRD1000W160D3600H5200, F.Cu at (133.0, 35.0)
- added C23: 104, Capacitor_SMD:C_0805_2012Metric, F.Cu at (349.6, 19.6)
- added C24: 333, Capacitor_SMD:C_0805_2012Metric, F.Cu at (349.6, 22.6)
- added C25: 102, Capacitor_SMD:C_0805_2012Metric, F.Cu at (349.6, 25.6)
- added C26: 104, Capacitor_SMD:C_0805_2012Metric, F.Cu at (349.6, 28.6)
- added C27: 102, Capacitor_SMD:C_0805_2012Metric, F.Cu at (349.6, 31.7)
- added C28: 102, Capacitor_SMD:C_0805_2012Metric, F.Cu at (349.6, 34.7)
- added C29: 104, Capacitor_SMD:C_0805_2012Metric, F.Cu at (321.2, 97.3)
- added C3: 104, Capacitor_SMD:C_0805_2012Metric, F.Cu at (340.7, 13.6)
- added C30: 102, Capacitor_SMD:C_0805_2012Metric, F.Cu at (354.1, 13.6)
- added C31: 102, Capacitor_SMD:C_0805_2012Metric, F.Cu at (354.1, 16.6)
- added C32: 104, Capacitor_SMD:C_0805_2012Metric, F.Cu at (354.1, 19.6)
- added C33: 104, Capacitor_SMD:C_0805_2012Metric, F.Cu at (354.1, 22.6)
- added C34: 104, Capacitor_SMD:C_0805_2012Metric, F.Cu at (354.1, 25.6)
- added C35: 2200uF/50V, Capacitor_THT:CP_Radial_D12.5mm_P7.50mm, F.Cu at (83.1, 25.6)
- added C36: 104, Capacitor_SMD:C_0805_2012Metric, F.Cu at (354.1, 28.6)
- added C37: 103, Capacitor_SMD:C_0805_2012Metric_Pad1.18x1.45mm_HandSolder, F.Cu at (348.9, 125.1)
- added C38: 103, Capacitor_SMD:C_0805_2012Metric_Pad1.18x1.45mm_HandSolder, F.Cu at (348.9, 128.1)
- added C39: 104, Capacitor_SMD:C_0805_2012Metric_Pad1.18x1.45mm_HandSolder, F.Cu at (348.9, 131.1)
- added C4: 102, Capacitor_SMD:C_0805_2012Metric_Pad1.18x1.45mm_HandSolder, F.Cu at (348.9, 122.1)
- added C40: 104, Capacitor_SMD:C_0805_2012Metric_Pad1.18x1.45mm_HandSolder, F.Cu at (348.9, 134.1)
- added C41: 104, Capacitor_SMD:C_0805_2012Metric_Pad1.18x1.45mm_HandSolder, F.Cu at (353.7, 116.0)
- added C42: 104, Capacitor_SMD:C_0805_2012Metric_Pad1.18x1.45mm_HandSolder, F.Cu at (353.7, 119.0)
- added C43: 10uF, Capacitor_SMD:C_0805_2012Metric_Pad1.18x1.45mm_HandSolder, F.Cu at (353.7, 122.1)
- added C44: 10uF, Capacitor_SMD:C_0805_2012Metric_Pad1.18x1.45mm_HandSolder, F.Cu at (353.7, 125.1)
- added C45: 470uF/25V, Capacitor_SMD:CP_Elec_10x12.5, F.Cu at (130.5, 86.0)
- added C46: 470uF/25V, Capacitor_SMD:CP_Elec_10x12.5, F.Cu at (119.0, 54.0)
- added C47: 104, Capacitor_SMD:C_0805_2012Metric_Pad1.18x1.45mm_HandSolder, F.Cu at (119.0, 64.0)
- added C48: 470uF/25V, Capacitor_SMD:CP_Elec_10x12.5, F.Cu at (146.0, 76.0)
- added C49: 470uF/25V, Capacitor_SMD:CP_Elec_10x12.5, F.Cu at (159.0, 77.0)
- added C5: 102, Capacitor_SMD:C_0805_2012Metric, F.Cu at (340.7, 16.6)
- added C50: 104, Capacitor_SMD:C_0805_2012Metric_Pad1.18x1.45mm_HandSolder, F.Cu at (151.0, 49.0)
- added C51: 1uF, Capacitor_SMD:C_0805_2012Metric, F.Cu at (354.1, 31.7)
- added C52: 220uF/50V, Capacitor_SMD:CP_Elec_10x12.5, F.Cu at (150.2, 91.0)
- added C53: 334, Capacitor_SMD:C_0805_2012Metric_Pad1.18x1.45mm_HandSolder, F.Cu at (163.6, 91.0)
- added C54: 104, Capacitor_SMD:C_0805_2012Metric_Pad1.18x1.45mm_HandSolder, F.Cu at (235.9, 109.5)
- added C55: 220uF/50V, Capacitor_SMD:CP_Elec_10x12.5, F.Cu at (237.8, 99.9)
- added C56: 102/1kV, Resistor_THT:R_Axial_DIN0207_L6.3mm_D2.5mm_P10.16mm_Horizontal, F.Cu at (244.2, 157.7)
- added C57: 104, Capacitor_SMD:C_0805_2012Metric_Pad1.18x1.45mm_HandSolder, F.Cu at (358.5, 119.0)
- added C58: 10uF, Capacitor_SMD:C_0805_2012Metric_Pad1.18x1.45mm_HandSolder, F.Cu at (358.5, 122.1)
- added C59: 10uF, Capacitor_SMD:C_0805_2012Metric_Pad1.18x1.45mm_HandSolder, F.Cu at (358.5, 125.1)
- added C6: 104, Capacitor_SMD:C_0805_2012Metric, F.Cu at (340.7, 19.6)
- added C60: 104, Capacitor_SMD:C_0805_2012Metric_Pad1.18x1.45mm_HandSolder, F.Cu at (329.1, 93.1)
- added C61: 104, Capacitor_SMD:C_0805_2012Metric_Pad1.18x1.45mm_HandSolder, F.Cu at (329.1, 96.1)
- added C7: 104, Capacitor_SMD:C_0805_2012Metric, F.Cu at (340.7, 22.6)
- added C8: 102, Capacitor_SMD:C_0805_2012Metric, F.Cu at (340.7, 25.6)
- added C9: 104, Capacitor_SMD:C_0805_2012Metric, F.Cu at (340.7, 28.6)
- added D1: SS16, Diode_SMD:D_3220_8050Metric_Pad2.65x5.15mm_HandSolder, F.Cu at (87.4, 81.5)
- added D2: SS16, Diode_SMD:D_3220_8050Metric_Pad2.65x5.15mm_HandSolder, F.Cu at (131.0, 60.0)
- added D3: ES1F-ES1J, Diode_SMD:D_2114_3652Metric_Pad1.85x3.75mm_HandSolder, F.Cu at (206.1, 63.1)
- added D4: ES1F-ES1J, Diode_SMD:D_2114_3652Metric_Pad1.85x3.75mm_HandSolder, F.Cu at (216.9, 63.1)
- added D5: ES1F-ES1J, Diode_SMD:D_2114_3652Metric_Pad1.85x3.75mm_HandSolder, F.Cu at (172.0, 83.0)
- added D6: SS16, Diode_SMD:D_3220_8050Metric_Pad2.65x5.15mm_HandSolder, F.Cu at (240.4, 92.3)
- added D7: SS16, Diode_SMD:D_3220_8050Metric_Pad2.65x5.15mm_HandSolder, F.Cu at (206.1, 138.7)
- added D8: BYV29X-500, inv24VLib:TO507P1020X460X2000-2, F.Cu at (91.0, 102.0)
- added D9: BYV29X-500, inv24VLib:TO507P1020X460X2000-2, F.Cu at (236.0, 132.0)
- added F1: 3544-2, inv24VLib:FUSE_3544-2, F.Cu at (237.8, 122.8)
- added F2: 3544-2, inv24VLib:FUSE_3544-2, F.Cu at (236.6, 138.7)
- added H1: MountingHole_Pad, MountingHole:MountingHole_4.3mm_M4_Pad_Via, F.Cu at (259.0, 26.0)
- added H2: MountingHole_Pad, MountingHole:MountingHole_4.3mm_M4_Pad_Via, F.Cu at (157.5, 26.0)
- added H3: MountingHole_Pad, MountingHole:MountingHole_4.3mm_M4_Pad_Via, F.Cu at (41.0, 26.0)
- added H4: MountingHole_Pad, MountingHole:MountingHole_4.3mm_M4_Pad_Via, F.Cu at (41.0, 152.0)
- added H5: MountingHole_Pad, MountingHole:MountingHole_4.3mm_M4_Pad_Via, F.Cu at (157.5, 152.0)
- added H6: MountingHole_Pad, MountingHole:MountingHole_4.3mm_M4_Pad_Via, F.Cu at (259.0, 152.0)
- added IC1: FSAM50SM60A, inv24VLib:DIP-32, F.Cu at (197.8, 53.6)
- added J1: 0705530003, genCtrlPCB_Lib:MOLEX_0705530039, F.Cu at (256.9, 96.8)
- added J10: Screw_Terminal_01x01, TerminalBlock_Wuerth:Wuerth_REDCUBE-THR_WP-THRBU_74650073_THR, F.Cu at (252.5, 139.3)
- added J12: Screw_Terminal_01x01, TerminalBlock_Wuerth:Wuerth_REDCUBE-THR_WP-THRBU_74650073_THR, F.Cu at (252.5, 115.8)
- added J2: Conn_01x02, Connector_Molex:Molex_KK-396_A-41791-0002_1x02_P3.96mm_Vertical, F.Cu at (307.5, 63.8)
- added J3: Conn_01x02, Connector_Molex:Molex_KK-396_A-41791-0002_1x02_P3.96mm_Vertical, F.Cu at (317.3, 63.8)
- added J7: Screw_Terminal_01x03, TerminalBlock_Dinkle:TerminalBlock_Dinkle_DT-55-B01X-03_P10.00mm, F.Cu at (253.5, 64.0)
- added L1: 100uH, Inductor_SMD:L_12x12mm_H8mm, F.Cu at (197.8, 154.5)
- added L2: 100uH, Inductor_SMD:L_12x12mm_H8mm, F.Cu at (130.0, 72.0)
- added L3: 100uH, Inductor_SMD:L_12x12mm_H8mm, F.Cu at (108.0, 86.0)
- added L4: 22uH, inv24VLib:IND_HCTI-10-20.0, F.Cu at (103.0, 58.0)
- added L5: 100uH, Inductor_SMD:L_12x12mm_H8mm, F.Cu at (236.6, 113.3)
- added PC1: TLP115A, Package_SO:MFSOP6-5_4.4x3.6mm_P1.27mm, F.Cu at (220.1, 101.2)
- added PC2: TLP115A, Package_SO:MFSOP6-5_4.4x3.6mm_P1.27mm, F.Cu at (222.0, 110.1)
- added Q1: IRFZ44NPBF, Package_TO_SOT_THT:TO-220-3_Vertical, F.Cu at (54.0, 98.0)
- added Q2: IRFZ44NPBF, Package_TO_SOT_THT:TO-220-3_Vertical, F.Cu at (43.9, 97.4)
- added Q3: ZXTN2010ZTA, Package_TO_SOT_SMD:SOT-89-3, F.Cu at (68.9, 106.9)
- added Q4: ZXTN2010ZTA, Package_TO_SOT_SMD:SOT-89-3, F.Cu at (61.3, 106.3)
- added Q5: ZXTP2012ZTA, Package_TO_SOT_SMD:SOT-89-3, F.Cu at (52.4, 106.3)
- added Q6: ZXTP2012ZTA, Package_TO_SOT_SMD:SOT-89-3, F.Cu at (44.2, 106.3)
- added R1: 10, Resistor_SMD:R_0805_2012Metric_Pad1.20x1.40mm_HandSolder, F.Cu at (306.8, 180.6)
- added R10: 2K, Resistor_SMD:R_0805_2012Metric, F.Cu at (335.2, 148.6)
- added R11: 5.6, Resistor_SMD:R_2010_5025Metric_Pad1.40x2.65mm_HandSolder, F.Cu at (330.7, 175.4)
- added R12: 5.6, Resistor_SMD:R_2010_5025Metric_Pad1.40x2.65mm_HandSolder, F.Cu at (330.7, 179.6)
- added R13: 5.6, Resistor_SMD:R_2010_5025Metric_Pad1.40x2.65mm_HandSolder, F.Cu at (330.7, 183.8)
- added R14: 22, Resistor_SMD:R_2010_5025Metric_Pad1.40x2.65mm_HandSolder, F.Cu at (330.7, 188.0)
- added R15: 22, Resistor_SMD:R_2010_5025Metric_Pad1.40x2.65mm_HandSolder, F.Cu at (330.7, 192.2)
- added R16: 22, Resistor_SMD:R_2010_5025Metric_Pad1.40x2.65mm_HandSolder, F.Cu at (330.7, 196.4)
- added R17: 1M/2W, Resistor_SMD:R_1206_3216Metric_Pad1.30x1.75mm_HandSolder, F.Cu at (337.5, 188.1)
- added R18: 1M/2W, Resistor_SMD:R_1206_3216Metric_Pad1.30x1.75mm_HandSolder, F.Cu at (337.5, 191.4)
- added R19: 1K, Resistor_SMD:R_0805_2012Metric_Pad1.20x1.40mm_HandSolder, F.Cu at (311.5, 183.6)
- added R2: 10, Resistor_SMD:R_0805_2012Metric_Pad1.20x1.40mm_HandSolder, F.Cu at (306.8, 183.6)
- added R20: 2K, Resistor_SMD:R_0805_2012Metric, F.Cu at (335.2, 151.5)
- added R21: 2K, Resistor_SMD:R_0805_2012Metric, F.Cu at (335.2, 154.5)
- added R22: 470, Resistor_SMD:R_0805_2012Metric, F.Cu at (339.6, 139.7)
- added R23: 390, Resistor_SMD:R_0805_2012Metric, F.Cu at (339.6, 142.7)
- added R24: 3.9K, Resistor_SMD:R_0805_2012Metric, F.Cu at (339.6, 145.6)
- added R25: 45, Resistor_SMD:R_0805_2012Metric, F.Cu at (339.6, 148.6)
- added R26: 4.7K, Resistor_SMD:R_0805_2012Metric, F.Cu at (339.6, 151.5)
- added R27: 4.7K, Resistor_SMD:R_0805_2012Metric, F.Cu at (339.6, 154.5)
- added R28: 4.7K, Resistor_SMD:R_0805_2012Metric, F.Cu at (344.0, 139.7)
- added R29: 100, Resistor_SMD:R_0805_2012Metric, F.Cu at (344.0, 142.7)
- added R3: 10K, Resistor_SMD:R_0805_2012Metric_Pad1.20x1.40mm_HandSolder, F.Cu at (306.8, 186.5)
- added R30: 100, Resistor_SMD:R_0805_2012Metric, F.Cu at (344.0, 145.6)
- added R31: 100, Resistor_SMD:R_0805_2012Metric, F.Cu at (344.0, 148.6)
- added R32: 100, Resistor_SMD:R_0805_2012Metric, F.Cu at (344.0, 151.5)
- added R33: 100, Resistor_SMD:R_0805_2012Metric, F.Cu at (344.0, 154.5)
- added R34: 100, Resistor_SMD:R_0805_2012Metric, F.Cu at (348.5, 139.7)
- added R35: 4.7K, Resistor_SMD:R_0805_2012Metric, F.Cu at (348.5, 142.7)
- added R36: 4.7K, Resistor_SMD:R_0805_2012Metric, F.Cu at (348.5, 145.6)
- added R37: 4.7K, Resistor_SMD:R_0805_2012Metric, F.Cu at (348.5, 148.6)
- added R38: 10K, Resistor_SMD:R_0805_2012Metric_Pad1.20x1.40mm_HandSolder, F.Cu at (311.5, 186.5)
- added R39: 2K, Resistor_SMD:R_0805_2012Metric_Pad1.20x1.40mm_HandSolder, F.Cu at (311.5, 189.5)
- added R4: 10K, Resistor_SMD:R_0805_2012Metric_Pad1.20x1.40mm_HandSolder, F.Cu at (306.8, 189.5)
- added R40: 10K, Resistor_SMD:R_0805_2012Metric_Pad1.20x1.40mm_HandSolder, F.Cu at (311.5, 192.4)
- added R41: 100, Resistor_SMD:R_0805_2012Metric_Pad1.20x1.40mm_HandSolder, F.Cu at (316.3, 180.6)
- added R42: 1K, Resistor_SMD:R_0805_2012Metric_Pad1.20x1.40mm_HandSolder, F.Cu at (315.0, 22.3)
- added R43: 120, Resistor_SMD:R_0805_2012Metric_Pad1.20x1.40mm_HandSolder, F.Cu at (315.0, 25.2)
- added R44: 4.7K, Resistor_SMD:R_0805_2012Metric_Pad1.20x1.40mm_HandSolder, F.Cu at (316.3, 183.6)
- added R45: 220, Resistor_SMD:R_0805_2012Metric_Pad1.20x1.40mm_HandSolder, F.Cu at (315.0, 28.2)
- added R46: 470, Resistor_SMD:R_0805_2012Metric_Pad1.20x1.40mm_HandSolder, F.Cu at (315.0, 31.1)
- added R47: 0, Resistor_SMD:R_0805_2012Metric_Pad1.20x1.40mm_HandSolder, F.Cu at (315.0, 34.1)
- added R48: 60, Resistor_SMD:R_0805_2012Metric_Pad1.20x1.40mm_HandSolder, F.Cu at (319.7, 22.3)
- added R49: 60, Resistor_SMD:R_0805_2012Metric_Pad1.20x1.40mm_HandSolder, F.Cu at (319.7, 25.2)
- added R5: 100, Resistor_SMD:R_0805_2012Metric_Pad1.20x1.40mm_HandSolder, F.Cu at (306.8, 192.4)
- added R50: 51.1K, Resistor_SMD:R_0805_2012Metric_Pad1.20x1.40mm_HandSolder, F.Cu at (319.7, 28.2)
- added R51: 6.04K, Resistor_SMD:R_0805_2012Metric_Pad1.20x1.40mm_HandSolder, F.Cu at (319.7, 31.1)
- added R52: 200K, Resistor_SMD:R_0805_2012Metric_Pad1.20x1.40mm_HandSolder, F.Cu at (319.7, 34.1)
- added R53: 1k, Resistor_SMD:R_0805_2012Metric_Pad1.20x1.40mm_HandSolder, F.Cu at (324.5, 22.3)
- added R54: 127K, Resistor_SMD:R_0805_2012Metric_Pad1.20x1.40mm_HandSolder, F.Cu at (324.5, 25.2)
- added R55: 10K, Resistor_SMD:R_0805_2012Metric_Pad1.20x1.40mm_HandSolder, F.Cu at (324.5, 28.2)
- added R56: 300K, Resistor_SMD:R_0805_2012Metric_Pad1.20x1.40mm_HandSolder, F.Cu at (324.5, 31.1)
- added R57: 10, Resistor_SMD:R_0805_2012Metric_Pad1.20x1.40mm_HandSolder, F.Cu at (316.3, 186.5)
- added R58: 10, Resistor_SMD:R_0805_2012Metric_Pad1.20x1.40mm_HandSolder, F.Cu at (316.3, 189.5)
- added R59: 22, Resistor_SMD:R_2010_5025Metric_Pad1.40x2.65mm_HandSolder, F.Cu at (322.8, 93.7)
- added R6: 100, Resistor_SMD:R_0805_2012Metric_Pad1.20x1.40mm_HandSolder, F.Cu at (311.5, 180.6)
- added R60: 470, Resistor_SMD:R_0805_2012Metric, F.Cu at (346.4, 71.2)
- added R61: 10K, Resistor_SMD:R_0805_2012Metric, F.Cu at (346.4, 74.2)
- added R62: 470, Resistor_SMD:R_0805_2012Metric, F.Cu at (346.4, 77.1)
- added R63: 10K, Resistor_SMD:R_0805_2012Metric, F.Cu at (346.4, 80.1)
- added R64: 10K, Resistor_SMD:R_0805_2012Metric, F.Cu at (346.4, 83.0)
- added R65: 10K, Resistor_SMD:R_0805_2012Metric, F.Cu at (346.4, 86.0)
- added R7: 2K, Resistor_SMD:R_0805_2012Metric, F.Cu at (335.2, 139.7)
- added R8: 2K, Resistor_SMD:R_0805_2012Metric, F.Cu at (335.2, 142.7)
- added R9: 2K, Resistor_SMD:R_0805_2012Metric, F.Cu at (335.2, 145.6)
- added RV1: ERZ-VF2M560, inv24VLib:VAR_ERZ-VF2M560, F.Cu at (222.0, 136.1)
- added RV2: ERZ-VF2M560, inv24VLib:VAR_ERZ-VF2M560, F.Cu at (252.5, 128.5)
- added RV3: ERZ-VF2M560, inv24VLib:VAR_ERZ-VF2M560, F.Cu at (222.6, 120.9)
- added RV4: ERZ-VF2M560, inv24VLib:VAR_ERZ-VF2M560, F.Cu at (247.4, 150.7)
- added T1: 1916_8p, genCtrlPCB_Lib:EE16_8_5_THT_H_9PIN_EXT__5280_, F.Cu at (203.6, 102.5)
- added TP1: TestPoint, TestPoint:TestPoint_Loop_D2.50mm_Drill1.0mm, F.Cu at (140.1, 90.4)
- added TP2: TestPoint, TestPoint:TestPoint_Loop_D2.50mm_Drill1.0mm, F.Cu at (116.0, 73.0)
- added TP3: TestPoint, TestPoint:TestPoint_Loop_D2.50mm_Drill1.0mm, F.Cu at (228.3, 82.8)
- added TP4: TestPoint, TestPoint:TestPoint_Loop_D2.50mm_Drill1.0mm, F.Cu at (246.7, 110.1)
- added U1: ESP32-DEVKITC-32D, inv24VLib:MODULE_ESP32-DEVKITC-32D, F.Cu at (95.6, 139.9)
- added U10: FOD817A, inv24VLib:PDIP4GW_709AH_ONS-M, F.Cu at (325.8, 73.4)
- added U11: ACT45B-220-2P-TL003, genCtrlPCB_Lib:FIL_ACT45B-220-2P-TL003, F.Cu at (224.5, 103.1)
- added U12: LM2576R-5.0, genCtrlPCB_Lib:VREG_TPS79625KTTR, F.Cu at (152.0, 62.0)
- added U13: FOD817A, inv24VLib:PDIP4GW_709AH_ONS-M, F.Cu at (325.8, 80.6)
- added U14: KIA7805AF, Package_TO_SOT_SMD:ATPAK-2, F.Cu at (239.1, 85.3)
- added U15: FOD817A, inv24VLib:PDIP4GW_709AH_ONS-M, F.Cu at (325.8, 87.9)
- added U2: LM2576R-5.0, genCtrlPCB_Lib:VREG_TPS79625KTTR, F.Cu at (224.5, 155.2)
- added U3: ACS712ELCTR30AT, inv24VLib:SOIC127P600X175-8N, F.Cu at (194.0, 23.7)
- added U4: ACS712ELCTR30AT, inv24VLib:SOIC127P600X175-8N, F.Cu at (207.4, 24.4)
- added U5: LM5160QPWPQ1, genCtrlPCB_Lib:SOP65P640X110-15N, F.Cu at (190.9, 120.2)
- added U6: ISO7340CDW, inv24VLib:SOIC127P1030X265-16N, F.Cu at (109.0, 104.0)
- added U7: ISO7340CDW, inv24VLib:SOIC127P1030X265-16N, F.Cu at (140.0, 112.0)
- added U8: AMC1300BDWVR, inv24VLib:SOIC127P1150X280-8N, F.Cu at (176.9, 112.0)
- added U9: TJA1040T, genCtrlPCB_Lib:SOIC127P600X175-8N, F.Cu at (226.4, 95.5)
- added X1: ~, inv24VLib:ee42208x8p, F.Cu at (40.6, 80.0)
- added ZD1: ZMM55C27, Diode_SMD:D_MiniMELF, F.Cu at (228.3, 97.4)
- added ZD2: ZMM55C27, Diode_SMD:D_MiniMELF, F.Cu at (223.9, 89.8)
- added ZD3: ZMM55C27, Diode_SMD:D_MiniMELF, F.Cu at (223.2, 86.0)
Other:
- board size 220 x 150 mm -> 237.5 x 150 mm

Commit message: fsam05 before change to NFA50460R4B
Parts:
- removed C57: 104, Capacitor_SMD:C_0805_2012Metric_Pad1.18x1.45mm_HandSolder
- removed C58, C59: 10uF, Capacitor_SMD:C_0805_2012Metric_Pad1.18x1.45mm_HandSolder
- removed R50: 51.1K, Resistor_SMD:R_0805_2012Metric_Pad1.20x1.40mm_HandSolder
- removed R51: 6.04K, Resistor_SMD:R_0805_2012Metric_Pad1.20x1.40mm_HandSolder
- removed R52: 200K, Resistor_SMD:R_0805_2012Metric_Pad1.20x1.40mm_HandSolder
- removed R54: 127K, Resistor_SMD:R_0805_2012Metric_Pad1.20x1.40mm_HandSolder
- removed R55: 10K, Resistor_SMD:R_0805_2012Metric_Pad1.20x1.40mm_HandSolder
- removed R56: 300K, Resistor_SMD:R_0805_2012Metric_Pad1.20x1.40mm_HandSolder
- removed T1: 1916_8p, genCtrlPCB_Lib:EE16_8_5_THT_H_9PIN_EXT__5280_
- added C62: 102, Capacitor_SMD:C_0805_2012Metric, F.Cu at (192.0, 34.0)
- added SW1: SW_DIP_x02, inv24VLib:PDIP4GW_709AH_ONS-M, F.Cu at (253.0, 73.0)
- C3: value 104 -> 470uF/25V; footprint Capacitor_SMD:C_0805_2012Metric -> Capacitor_SMD:CP_Elec_10x12.5
- C4: value 102 -> 104
- C42: value 104 -> 470uF/25V; footprint Capacitor_SMD:C_0805_2012Metric_Pad1.18x1.45mm_HandSolder -> Capacitor_SMD:CP_Elec_10x12.5
- C43: value 10uF -> 104
- C44: value 10uF -> 470uF/25V; footprint Capacitor_SMD:C_0805_2012Metric_Pad1.18x1.45mm_HandSolder -> Capacitor_SMD:CP_Elec_10x12.5
- C51: value 1uF -> 104; footprint Capacitor_SMD:C_0805_2012Metric -> Capacitor_SMD:C_0805_2012Metric_Pad1.18x1.45mm_HandSolder
- IC1: moved to B.Cu
- Q1, Q2: footprint Package_TO_SOT_THT:TO-220-3_Vertical -> Package_TO_SOT_THT:TO-220-3_Horizontal_TabUp; moved to B.Cu
- U5: value LM5160QPWPQ1 -> ~; footprint genCtrlPCB_Lib:SOP65P640X110-15N -> Library:ewDCDC24_1505d
- moved C33 302.6 mm to (56.0, 75.0)
- moved C36 301.1 mm to (56.0, 71.0)
- moved C21 293.3 mm to (62.0, 74.0)
- moved C19 293.0 mm to (56.0, 82.0)
- moved R64 291.4 mm to (56.0, 59.0)
- moved R39 285.1 mm to (56.0, 63.0)
- moved BX1 284.9 mm to (94.0, 27.0)
- moved R65 284.5 mm to (62.0, 82.0)
- moved BX4 284.1 mm to (102.0, 26.0)
- moved R41 284.0 mm to (56.0, 67.0)
- moved BX2 282.1 mm to (102.0, 23.0)
- moved R8 281.9 mm to (65.1, 62.3), turned to 90 degrees
- moved R9 281.6 mm to (65.1, 66.1), turned to -90 degrees
- moved R10 280.7 mm to (68.1, 62.3), turned to 90 degrees
- moved R21 279.1 mm to (68.0, 74.0)
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Connections:
- C3 pad 1: Net-(U5-BST) -> +8VP_IN
- C3 pad 2: Net-(C3-Pad2) -> GND1
- C4 pad 1: Net-(C4-Pad1) -> +8VP_IN
- C4 pad 2: Net-(C4-Pad2) -> GND1
- C42 pad 1: Net-(C4-Pad2) -> 15V_H_IN
- C42 pad 2: Net-(U5-FB) -> GND2
- C43 pad 1: GND -> 15V_H_IN
- C43 pad 2: Net-(C4-Pad1) -> GND2
- C44 pad 1: GND -> +24V
- C44 pad 2: Net-(C4-Pad1) -> GND
- C48 pad 1: +5V -> +5VP
- C49 pad 1: +5V -> +5VP
- C50 pad 2: +5V -> +5VP
- C51 pad 1: GND -> +24V
- C51 pad 2: Net-(U5-FPWM) -> GND
- L2 pad 2: +5V -> +5VP
- R53 pad 2: +5V -> +5VP
- TP1 pad 1: +5V -> +5VP
- U12 pad 4: +5V -> +5VP
- U5 pad 1: GND -> +24V
- U5 pad 10: Net-(U5-FPWM) -> unconnected-(U5-nOut2-Pad10)
- U5 pad 3: +24V -> unconnected-(U5-NC1-Pad3)
- U5 pad 4: Net-(U5-EN/UVLO) -> unconnected-(U5-NC2-Pad4)
- U5 pad 5: Net-(U5-RON) -> unconnected-(U5-Vout1-Pad5)
- U5 pad 6: Net-(U5-SS) -> +8VP_IN
- U5 pad 7: unconnected-(U5-NC-Pad7) -> GND1
- U5 pad 8: Net-(U5-FPWM) -> 15V_H_IN
- U5 pad 9: Net-(U5-FB) -> GND2
- X1 pad 10: H+15V -> unconnected-(X1-Pad10)
- X1 pad 9: GND2 -> unconnected-(X1-Pad9)
Other:
- outline, holes or cut-outs redrawn

Commit message: before delete isolation
Parts:
- removed C13, C14, C15: 22uF/25V, Capacitor_SMD:C_0805_2012Metric
- removed C16, C17, C18, C23: 104, Capacitor_SMD:C_0805_2012Metric
- removed C24: 333, Capacitor_SMD:C_0805_2012Metric
- removed C25: 102, Capacitor_SMD:C_0805_2012Metric
- removed D3, D4, D5: ES1F-ES1J, Diode_SMD:D_2114_3652Metric_Pad1.85x3.75mm_HandSolder
- removed IC1: FSAM50SM60A, inv24VLib:DIP-32
- removed R11, R12, R13: 5.6, Resistor_SMD:R_2010_5025Metric_Pad1.40x2.65mm_HandSolder
- removed R14, R15, R16: 22, Resistor_SMD:R_2010_5025Metric_Pad1.40x2.65mm_HandSolder
- removed R23: 390, Resistor_SMD:R_0805_2012Metric
- removed R24: 3.9K, Resistor_SMD:R_0805_2012Metric
- removed R25: 45, Resistor_SMD:R_0805_2012Metric
- removed R26, R27, R28, R35, R36, R37: 4.7K, Resistor_SMD:R_0805_2012Metric
