File: inv24to120V.kicad_sch (KiCad schematic)
At the start: 133 parts, among them IC1 FSAM50SM60A, J1 Conn_02x13_Odd_Even_MountingP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, J10 Screw_Terminal_01x01, J11 Screw_Terminal_01x01, J12 Screw_Terminal_01x01, J2 Conn_02x13_Odd_Even_MountingP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, J3 Screw_Terminal_01x01, J4 Conn_02x05_Odd_Even_MountingP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, J5 Screw_Terminal_01x02, J6 Screw_Terminal_01x03, J7 Screw_Terminal_01x03, J8 Screw_Terminal_01x03, J9 Screw_Terminal_01x02, K1 J0971CS5VDC.45, Q1 IRFZ44NPBF, Q2 IRFZ44NPBF, Q3 2SC1815, Q4 2SC1815, Q5 2SA1015, Q6 2SA1015, Q7 2SC1815, U1 ESP32-DEVKITC-32D, U10 PC817, U2 LM2576HVT-5, U3 ACS712ELCTR30AT, U4 ACS712ELCTR30AT, U5 LM2576HVT-5, U6 ISO7340CDW, U7 ISO7340CDW, U8 AMC1300BDWVR, U9 PC817

Commit message: for 220V fan control
Parts:
- removed BX1, BX2: 0, Resistor_THT:R_Axial_DIN0207_L6.3mm_D2.5mm_P10.16mm_Horizontal, symbol bead:bead
- removed C3: 470uF/50V, Capacitor_THT:CP_Radial_D8.0mm_P5.00mm, symbol Device:C_Polarized
- removed C4: 100uF/50V, Capacitor_THT:CP_Radial_D8.0mm_P5.00mm, symbol Device:C_Polarized
- removed D7: 1N4002, Diode_THT:D_DO-41_SOD81_P10.16mm_Horizontal, symbol Diode:1N4002
- removed J1, J2: Conn_02x13_Odd_Even_MountingPin, Connector_IDC:IDC-Header_2x13_P2.54mm_Vertical, symbol Connector_Generic_MountingPin:Conn_02x13_Odd_Even_MountingPin
- removed J4: Conn_02x05_Odd_Even_MountingPin, Connector_IDC:IDC-Header_2x05_P2.54mm_Vertical, symbol Connector_Generic_MountingPin:Conn_02x05_Odd_Even_MountingPin
- removed J6: Screw_Terminal_01x03, TerminalBlock_Phoenix:TerminalBlock_Phoenix_MKDS-1,5-3-5.08_1x03_P5.08mm_Horizontal, symbol Connector:Screw_Terminal_01x03
- removed J8: Screw_Terminal_01x03, TerminalBlock_Phoenix:TerminalBlock_Phoenix_MKDS-1,5-3_1x03_P5.00mm_Horizontal, symbol Connector:Screw_Terminal_01x03
- removed J9: Screw_Terminal_01x02, TerminalBlock_Phoenix:TerminalBlock_Phoenix_MKDS-1,5-2-5.08_1x02_P5.08mm_Horizontal, symbol Connector:Screw_Terminal_01x02
- removed K1: J0971CS5VDC.45, inv24VLib:RELAY_J0971CS5VDC.45, symbol J0971CS5VDC.45:J0971CS5VDC.45
- removed Q7: 2SC1815, Package_TO_SOT_THT:TO-92_Inline, symbol Transistor_BJT:2SC1815
- removed U2, U5: LM2576HVT-5, Package_TO_SOT_THT:TO-220-5_Vertical, symbol Regulator_Switching:LM2576HVT-5
- removed U9: PC817, Package_DIP:DIP-4_W7.62mm, symbol Isolator:PC817
- added BC1, BC2, C39, C40, C41, C42, C47, C50, C54, C57: 104, Capacitor_SMD:C_0805_2012Metric_Pad1.18x1.45mm_HandSolder, symbol Device:C
- added C19, C3: 104, Capacitor_SMD:C_0805_2012Metric, symbol Device:C
- added C38: 103, Capacitor_SMD:C_0805_2012Metric_Pad1.18x1.45mm_HandSolder, symbol Device:C
- added C4: 102, Capacitor_SMD:C_0805_2012Metric_Pad1.18x1.45mm_HandSolder, symbol Device:C
- added C43, C44, C58, C59: 10uF, Capacitor_SMD:C_0805_2012Metric_Pad1.18x1.45mm_HandSolder, symbol Device:C
- added C45, C46, C48, C49: 470uF/25V, Capacitor_SMD:CP_Elec_10x12.5, symbol Device:C_Polarized
- added C51: 1uF, Capacitor_SMD:C_0805_2012Metric, symbol Device:C
- added C52, C55: 220uF/50V, Capacitor_SMD:CP_Elec_10x12.5, symbol Device:C_Polarized
- added C53: 334, Capacitor_SMD:C_0805_2012Metric_Pad1.18x1.45mm_HandSolder, symbol Device:C
- added C56: 102/1kV, Resistor_THT:R_Axial_DIN0207_L6.3mm_D2.5mm_P10.16mm_Horizontal, symbol Device:C
- added D7: SS16, Diode_SMD:D_3220_8050Metric_Pad2.65x5.15mm_HandSolder, symbol Diode:1N5822
- added H1, H2, H3, H4, H5, H6: MountingHole_Pad, MountingHole:MountingHole_4.3mm_M4_Pad_Via, symbol Mechanical:MountingHole_Pad
- added J1: 0705530003, 0705530003:MOLEX_0705530003, symbol 0705530003:0705530003
- added L5: 100uH, Inductor_SMD:L_12x12mm_H8mm, symbol Device:L
- added PC1, PC2: TLP115A, Package_SO:MFSOP6-5_4.4x3.6mm_P1.27mm, symbol Isolator:TLP137
- added R38: 10K, Resistor_THT:R_Axial_DIN0207_L6.3mm_D2.5mm_P10.16mm_Horizontal, symbol Device:R
- added R39: 2K, Resistor_THT:R_Axial_DIN0207_L6.3mm_D2.5mm_P10.16mm_Horizontal, symbol Device:R
- added R41: 100, Resistor_THT:R_Axial_DIN0207_L6.3mm_D2.5mm_P10.16mm_Horizontal, symbol Device:R
- added R43: 120, Resistor_SMD:R_0805_2012Metric_Pad1.20x1.40mm_HandSolder, symbol Device:R
- added R49: 60, Resistor_SMD:R_0805_2012Metric_Pad1.20x1.40mm_HandSolder, symbol Device:R
- added R50: 51.1K, Resistor_SMD:R_0805_2012Metric_Pad1.20x1.40mm_HandSolder, symbol Device:R
- added R51: 6.04K, Resistor_SMD:R_0805_2012Metric_Pad1.20x1.40mm_HandSolder, symbol Device:R
- added R52: 200K, Resistor_SMD:R_0805_2012Metric_Pad1.20x1.40mm_HandSolder, symbol Device:R
- added R53: 1k, Resistor_SMD:R_0805_2012Metric_Pad1.20x1.40mm_HandSolder, symbol Device:R
- added R54: 127K, Resistor_SMD:R_0805_2012Metric_Pad1.20x1.40mm_HandSolder, symbol Device:R
- added R55: 10K, Resistor_SMD:R_0805_2012Metric_Pad1.20x1.40mm_HandSolder, symbol Device:R
- added R56: 300K, Resistor_SMD:R_0805_2012Metric_Pad1.20x1.40mm_HandSolder, symbol Device:R
- added T1: 1916_8p, 750313739:EE16_8_5_THT_H_9PIN_EXT__5280_, symbol 750313739:750313739
- added TP1, TP2, TP3, TP4: TestPoint, TestPoint:TestPoint_Loop_D2.50mm_Drill1.0mm, symbol Connector:TestPoint
- added U11: ACT45B-220-2P-TL003, ACT45B-220-2P-TL003:FIL_ACT45B-220-2P-TL003, symbol ACT45B-220-2P-TL003:ACT45B-220-2P-TL003
- added U12, U2: LM2576R-5.0, LM2576S-12_NOPB:VREG_TPS79625KTTR, symbol LM2576S-12_NOPB:LM2576S-12_NOPB
- added U14: KIA7805AF, Package_TO_SOT_SMD:ATPAK-2, symbol Regulator_Linear:L7805
- added U5: LM5160QPWPQ1, LM5160QPWPQ1:SOP65P640X110-15N, symbol LM5160QPWPQ1:LM5160QPWPQ1
- added U9: TJA1040T, TJA1040T:SOIC127P600X175-8N, symbol TJA1040T:TJA1040T
- added ZD1, ZD2, ZD3: ZMM55C27, Diode_SMD:D_MiniMELF, symbol Diode:ZMMxx
- C37: value 104 -> 103; footprint Capacitor_SMD:C_0805_2012Metric -> Capacitor_SMD:C_0805_2012Metric_Pad1.18x1.45mm_HandSolder
- D1, D2, D6: value 1N5822 -> SS16; footprint Diode_THT:D_DO-201AD_P15.24mm_Horizontal -> Diode_SMD:D_3220_8050Metric_Pad2.65x5.15mm_HandSolder
- L2, L3: footprint Inductor_THT:L_Radial_D10.0mm_P5.00mm_Neosid_SD12k_style3 -> Inductor_SMD:L_12x12mm_H8mm
- R42: value 4.7K -> 1K; footprint Resistor_THT:R_Axial_DIN0207_L6.3mm_D2.5mm_P10.16mm_Horizontal -> Resistor_SMD:R_0805_2012Metric_Pad1.20x1.40mm_HandSolder
- R45: value 470 -> 220; footprint Resistor_THT:R_Axial_DIN0207_L6.3mm_D2.5mm_P10.16mm_Horizontal -> Resistor_SMD:R_0805_2012Metric_Pad1.20x1.40mm_HandSolder
- R46: value 4.7K -> 470; footprint Resistor_THT:R_Axial_DIN0207_L6.3mm_D2.5mm_P10.16mm_Horizontal -> Resistor_SMD:R_0805_2012Metric_Pad1.20x1.40mm_HandSolder
- R47: value 470 -> 0; footprint Resistor_THT:R_Axial_DIN0207_L6.3mm_D2.5mm_P10.16mm_Horizontal -> Resistor_SMD:R_0805_2012Metric_Pad1.20x1.40mm_HandSolder
- R48: value 4.7K -> 60; footprint Resistor_THT:R_Axial_DIN0207_L6.3mm_D2.5mm_P10.16mm_Horizontal -> Resistor_SMD:R_0805_2012Metric_Pad1.20x1.40mm_HandSolder
Connections:
- net 150V_OUT1 is gone; now on net VBUS: D8.2 (A), X1.15, X1.16
- net FAULT_IPM2 is gone; now on net FAULT_IPM: R44.2, U10.4
- net GNDPWR1 is gone; now on net GNDPWR: J10.1 (Pin_1), R19.1, U8.3 (INN), X1.12, X1.13
- net I_Uphase2 is gone; now on net I_Uphase: R7.1, R9.2
- net I_Vphase2 is gone; now on net I_Vphase: R10.2, R8.1
- net TEMPERATURE_IPM2 is gone; now on net TEMPERATURE_IPM: BX6.1, C34.2, R40.2
- net UH2 is gone; now on net UH1: R29.1
- net UL2 is gone; now on net UL1: R32.1
- net VH2 is gone; now on net VH1: R30.1
- net VL2 is gone; now on net VL1: R33.1
- net VTH_IPM2 is gone; now on net VTH_IPM: IC1.24 (VTH)
- net WH2 is gone; now on net WH1: R31.1
- net WL2 is gone; now on net WL1: R34.1
- net +15V: no longer L3.2
- net +24V: now also C58.2, C59.2, R39.2, R54.2, R56.2, U2.1 (VIN), U5.3 (VIN)
- net +3.3V: now also R42.1, PC2.6, R43.2; no longer R48.2
- net +5V: now also L2.2, C48.1, C49.1, C50.2, R53.2, TP1.1, U12.4 (FB), U2.4 (FB)
- net +5VP: no longer L2.2
- net ANALOG_CMD: no longer R42.1
- net DIGITAL_CMD: no longer C37.2, R48.1
- net GND: now also C19.1, C43.1, C44.1, C51.1, C56.1, C57.2, C58.1, C59.1, D7.2 (A), PC2.4, R41.1, R52.1, R55.1, U2.3 (GND), U2.5 (ON/OFF), U2.6 (GND), U5.1 (AGND), U5.15 (EXP), U5.2 (PGND); no longer D1.2 (A), R46.2, R47.2
- net GND2: now also C45.2, C46.2, C47.1, C48.2, C49.2, C50.1, R53.1, T1.7, U12.3 (GND), U12.5 (ON/OFF), U12.6 (GND)
- net GNDPWR: now also IC1.16 (COM(H))
- net H+15V: no longer D6.2 (A)
- net RELAY_TRIP: no longer R45.1
- net +5P: now reaches R45.2, R46.1
- net +5P: now also BC1.2, BC2.2, C38.2, C54.2, C55.1, J1.1, PC1.6, TP4.1, U14.3 (OUT), U9.3 (VCC)
- net RX_CAN: now reaches R42.2
- net RX_CAN: now also C37.2, PC2.5
- net at D6.1 (K): now also L5.1, TP3.1; no longer L3.1
- net at L1.1: now also D7.1 (K), U2.2 (OUT); no longer D1.1 (K)
- net at R47.1: now also R48.1, C39.1, R49.1
- net at D2.1 (K), L2.1: now also U12.2 (OUT)
- net VDC_IN: now reaches U1.J2-8 (IO33)
- net VDC_IN: now also C19.2, R38.2
- net VTH_IPM1 renamed VTH_IPM
- new net: C56.2, H1.1
- new net: C45.1, C46.1, C47.2, L3.2, TP2.1, U12.1 (VIN)
- new net: PC1.1, R43.1
- new net: R56.1, U5.5 (RON)
- new net: C40.1, J1.4, R49.2, U11.3, ZD3.1 (K)
- new net: ZD1.2 (A), ZD2.2 (A), ZD3.2 (A)
- new net: U11.1, U9.7 (CANH)
- new net: U11.2, U9.6 (CANL)
- new net: C41.1, J1.3, R48.2, U11.4, ZD1.1 (K)
- new net: R38.1, R39.1, R41.2
- new net: C4.1, C43.2, C44.2, R51.1, T1.1
- new net: C4.2, C42.1, R50.1
- new net: C3.1, U5.11 (BST)
- new net: C3.2, R50.2, T1.8, U5.12 (SW), U5.13 (SW)
- new net: C42.2, R51.2, R52.2, U5.9 (FB)
- new net: C51.2, U5.10 (VCC), U5.8 (FPWM)
- new net: R47.2, U9.5 (SPLIT)
- new net: PC1.5, R46.2, U9.1 (TXD)
- new net: PC2.3, U9.4 (RXD)
- new net: R54.1, R55.2, U5.4 (EN/UVLO)
- new net: C57.1, U5.6 (SS)
- new net: D1.1 (K), L3.1
- new net: PC2.1, R45.1
- new net +8VP_IN: D6.2 (A), T1.3
- new net +BATT: C52.1, C53.2, L5.2, U14.1 (IN)
- new net 15V_H_IN: D1.2 (A), T1.5
- new net GND1: BC1.1, BC2.1, C38.1, C39.2, C40.2, C41.2, C52.2, C53.1, C54.1, C55.2, J1.2, PC1.4, T1.2, U14.2 (GND), U9.2 (GND), U9.8 (STB), ZD2.1 (K)
- new net TX_CAN: PC1.3

Commit message: start place parts
Parts:
- removed BX5, BX6: 0, Resistor_THT:R_Axial_DIN0207_L6.3mm_D2.5mm_P10.16mm_Horizontal, symbol bead:bead
- removed J11, J3: Screw_Terminal_01x01, TerminalBlock_Wuerth:Wuerth_REDCUBE-THR_WP-THRBU_74650073_THR, symbol Connector:Screw_Terminal_01x01
- removed J5: Screw_Terminal_01x02, TerminalBlock_Dinkle:TerminalBlock_Dinkle_DT-55-B01X-02_P10.00mm, symbol Connector:Screw_Terminal_01x02
- removed Q4: 2SC1815, Package_TO_SOT_THT:TO-92_Inline, symbol Transistor_BJT:2SC1815
- removed Q6: 2SA1015, Package_TO_SOT_THT:TO-92_Inline, symbol Transistor_BJT:2SA1015
- added BX1, BX2: BLM31KN801SH1L, Resistor_SMD:R_1206_3216Metric_Pad1.30x1.75mm_HandSolder, symbol bead:bead
- added C60, C61: 104, Capacitor_SMD:C_0805_2012Metric_Pad1.18x1.45mm_HandSolder, symbol Device:C
- added J2, J3: Conn_01x02, Connector_Molex:Molex_KK-396_A-41791-0002_1x02_P3.96mm_Vertical, symbol Connector_Generic:Conn_01x02
- added Q4: ZXTN2010ZTA, Package_TO_SOT_SMD:SOT-89-3, symbol Transistor_BJT:2SD1047
- added Q6: ZXTP2012ZTA, Package_TO_SOT_SMD:SOT-89-3, symbol Transistor_BJT:BCP51
- added R57, R58: 10, Resistor_SMD:R_0805_2012Metric_Pad1.20x1.40mm_HandSolder, symbol Device:R
- added R59: 22, Resistor_SMD:R_2010_5025Metric_Pad1.40x2.65mm_HandSolder, symbol Device:R
- added R60, R62: 470, Resistor_SMD:R_0805_2012Metric, symbol Device:R
- added R61, R63, R64, R65: 10K, Resistor_SMD:R_0805_2012Metric, symbol Device:R
- added RV1, RV2, RV3, RV4: ERZ-VF2M560, inv24VLib:VAR_ERZ-VF2M560, symbol ERZ-VF2M560:ERZ-VF2M560
- added U13, U15: FOD817A, inv24VLib:PDIP4GW_709AH_ONS-M, symbol Isolator:PC817
- BX3, BX4: value 0 -> BLM31KN801SH1L; footprint Resistor_THT:R_Axial_DIN0207_L6.3mm_D2.5mm_P10.16mm_Horizontal -> Resistor_SMD:R_1206_3216Metric_Pad1.30x1.75mm_HandSolder
- C1: value 100uF/50V -> 2200uF/50V; footprint Capacitor_THT:CP_Radial_D8.0mm_P5.00mm -> Capacitor_THT:CP_Radial_D12.5mm_P7.50mm
- C2: value 100uF/50V -> 470uF/25V; footprint Capacitor_THT:CP_Radial_D8.0mm_P5.00mm -> Capacitor_SMD:CP_Elec_10x12.5
- C29: value 102 -> 104
- C35: value 47uF/50V -> 2200uF/50V; footprint Capacitor_THT:CP_Radial_D8.0mm_P5.00mm -> Capacitor_THT:CP_Radial_D12.5mm_P7.50mm
- D3, D4, D5: value 1N4937 -> ES1F-ES1J; footprint Diode_THT:D_DO-35_SOD27_P10.16mm_Horizontal -> Diode_SMD:D_2114_3652Metric_Pad1.85x3.75mm_HandSolder
- J1: footprint 0705530003:MOLEX_0705530003 -> genCtrlPCB_Lib:MOLEX_0705530039
- L1: footprint Inductor_THT:L_Radial_D10.0mm_P5.00mm_Neosid_SD12k_style3 -> Inductor_SMD:L_12x12mm_H8mm
- Q3: value 2SC1815 -> ZXTN2010ZTA; footprint Package_TO_SOT_THT:TO-92_Inline -> Package_TO_SOT_SMD:SOT-89-3; symbol Transistor_BJT:2SC1815 -> Transistor_BJT:2SD1047
- Q5: value 2SA1015 -> ZXTP2012ZTA; footprint Package_TO_SOT_THT:TO-92_Inline -> Package_TO_SOT_SMD:SOT-89-3; symbol Transistor_BJT:2SA1015 -> Transistor_BJT:BCP51
- R1, R19, R2, R3, R38, R39, R4, R40, R41, R44, R5, R6: footprint Resistor_THT:R_Axial_DIN0207_L6.3mm_D2.5mm_P10.16mm_Horizontal -> Resistor_SMD:R_0805_2012Metric_Pad1.20x1.40mm_HandSolder
- R11, R12, R13: footprint Resistor_THT:R_Axial_DIN0207_L6.3mm_D2.5mm_P10.16mm_Horizontal -> Resistor_SMD:R_2010_5025Metric_Pad1.40x2.65mm_HandSolder
- R14, R15, R16: value 20 -> 22; footprint Resistor_THT:R_Axial_DIN0207_L6.3mm_D2.5mm_P10.16mm_Horizontal -> Resistor_SMD:R_2010_5025Metric_Pad1.40x2.65mm_HandSolder
- R17, R18: footprint Resistor_THT:R_Axial_DIN0414_L11.9mm_D4.5mm_P15.24mm_Horizontal -> Resistor_SMD:R_1206_3216Metric_Pad1.30x1.75mm_HandSolder
- T1: footprint 750313739:EE16_8_5_THT_H_9PIN_EXT__5280_ -> genCtrlPCB_Lib:EE16_8_5_THT_H_9PIN_EXT__5280_
- U10: value PC817 -> FOD817A; footprint Package_DIP:DIP-4_W7.62mm -> inv24VLib:PDIP4GW_709AH_ONS-M
- U11: footprint ACT45B-220-2P-TL003:FIL_ACT45B-220-2P-TL003 -> genCtrlPCB_Lib:FIL_ACT45B-220-2P-TL003
- U12, U2: footprint LM2576S-12_NOPB:VREG_TPS79625KTTR -> genCtrlPCB_Lib:VREG_TPS79625KTTR
- U5: footprint LM5160QPWPQ1:SOP65P640X110-15N -> genCtrlPCB_Lib:SOP65P640X110-15N
- U9: footprint TJA1040T:SOIC127P600X175-8N -> genCtrlPCB_Lib:SOIC127P600X175-8N
Connections:
- net +24V: now also C29.2, C35.1, R59.2, RV1.2, RV2.2, RV3.2; no longer D9.1 (K)
- net +3.3V: now also R64.1, R65.1
- net +5P: now also J2.1 (Pin_1), J3.1 (Pin_1)
- net +5V: now also Q3.2 (C), BX1.1, Q4.2 (C); no longer BX4.1, Q5.1 (E)
- net GND: now also C29.1, C35.2, Q5.2 (C), BX2.1, C60.1, C61.1, Q6.2 (C), RV1.1, U13.3, U15.3; no longer Q3.1 (E)
- net GND1: now also R61.2, R63.2, U13.2, U15.2
- net GND2: no longer C29.1
- net GNDPWR: no longer J10.1 (Pin_1)
- net IN_WH: no longer C29.2
- net TEMPERATURE_IPM: now also BX4.1
- net VBUS: now also L4.1, R17.2; no longer D8.2 (A), X1.15, X1.16
- net VTH_IPM: now also BX1.2; no longer BX4.2, C35.1
- net Earth: now reaches C56.2, H1.1
- net Earth: now also H2.1, H3.1, H4.1, H5.1, H6.1, RV4.1
- net at C33.1: now also BX2.2; no longer C35.2
- net at R2.1: now also Q4.3 (E)
- net at R6.2: now also Q4.1 (B), Q6.1 (B)
- net at C14.1, C17.1, IC1.18 (VB(V)): now also D3.1 (K); no longer D4.1 (K)
- net at C13.1, C16.1, IC1.22 (VB(W)): now also D4.1 (K); no longer D3.1 (K)
- net at Q2.1 (G), R2.2, R4.2: now also R58.2
- net DIN_A: now reaches U1.J3-13 (IO4)
- net DIN_A: now also C60.2, R64.2, U13.4
- net DIN_B: now reaches U1.J3-14 (IO0)
- net DIN_B: now also C61.2, R65.2, U15.4
- net at IC1.25 (RTH): now also BX4.2
- net at Q1.1 (G), R1.2, R3.2: now also R57.2
- net at F1.1_1, F1.1_2: now also J12.1 (Pin_1)
- net at F2.1_1, F2.1_2: now also J10.1 (Pin_1)
- new net: D9.1 (K), R59.1
- new net: RV2.1, RV3.1, RV4.2
- new net: R62.1, R63.1, U15.1
- new net: Q5.3 (E), R57.1
- new net: Q3.1 (B), Q5.1 (B), R5.2
- new net: J3.2 (Pin_2), R62.2
- new net: Q3.3 (E), R1.1
- new net: R60.1, R61.1, U13.1
- new net: Q6.3 (E), R58.1
- new net: J2.2 (Pin_2), R60.2
- new net 150V_OUT: D8.2 (A), X1.15, X1.16
- no-connect marks 0 -> 13
Other:
- moved on the sheet: C22, C33, C36, D7, D9, H2, H3, H4, H5, H6, J10, J12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

Commit message: fsam05 before change to NFA50460R4B
Parts:
- removed C3: 104, Capacitor_SMD:C_0805_2012Metric, symbol Device:C
- removed C42, C57: 104, Capacitor_SMD:C_0805_2012Metric_Pad1.18x1.45mm_HandSolder, symbol Device:C
- removed C44, C58, C59: 10uF, Capacitor_SMD:C_0805_2012Metric_Pad1.18x1.45mm_HandSolder, symbol Device:C
- removed R50: 51.1K, Resistor_SMD:R_0805_2012Metric_Pad1.20x1.40mm_HandSolder, symbol Device:R
- removed R51: 6.04K, Resistor_SMD:R_0805_2012Metric_Pad1.20x1.40mm_HandSolder, symbol Device:R
- removed R52: 200K, Resistor_SMD:R_0805_2012Metric_Pad1.20x1.40mm_HandSolder, symbol Device:R
- removed R54: 127K, Resistor_SMD:R_0805_2012Metric_Pad1.20x1.40mm_HandSolder, symbol Device:R
- removed R55: 10K, Resistor_SMD:R_0805_2012Metric_Pad1.20x1.40mm_HandSolder, symbol Device:R
- removed R56: 300K, Resistor_SMD:R_0805_2012Metric_Pad1.20x1.40mm_HandSolder, symbol Device:R
- removed T1: 1916_8p, genCtrlPCB_Lib:EE16_8_5_THT_H_9PIN_EXT__5280_, symbol 750313739:750313739
- removed U5: LM5160QPWPQ1, genCtrlPCB_Lib:SOP65P640X110-15N, symbol LM5160QPWPQ1:LM5160QPWPQ1
- added C3, C42, C44: 470uF/25V, Capacitor_SMD:CP_Elec_10x12.5, symbol Device:C_Polarized
- added C62: 102, Capacitor_SMD:C_0805_2012Metric, symbol Device:C
- added SW1: SW_DIP_x02, inv24VLib:PDIP4GW_709AH_ONS-M, symbol Switch:SW_DIP_x02
- added U5: ~, Library:ewDCDC24_1505d, symbol ewDCDC_24_1508d:con24_1508d
- C4: value 102 -> 104
- C43: value 10uF -> 104
- C51: value 1uF -> 104; footprint Capacitor_SMD:C_0805_2012Metric -> Capacitor_SMD:C_0805_2012Metric_Pad1.18x1.45mm_HandSolder
- Q1, Q2: footprint Package_TO_SOT_THT:TO-220-3_Vertical -> Package_TO_SOT_THT:TO-220-3_Horizontal_TabUp
Connections:
- net +24V: now also C51.1, C44.1, U5.1 (VIN1)
- net +5V: no longer C48.1, C49.1, C50.2, L2.2, R53.2, TP1.1, U12.4 (FB)
- net +5VP: now also C48.1, C49.1, C50.2, L2.2, R53.2, TP1.1, U12.4 (FB)
- net +8VP_IN: now also C4.1, C3.1, U5.6 (GND_1)
- net 15V_H_IN: now also C43.1, C42.1, U5.8 (Vout2)
- net DIN_A: now also SW1.4
- net DIN_B: now also SW1.3
- net GND: now also C51.2, C44.2, SW1.1, SW1.2, U5.2 (IN_GND); no longer C43.1, C51.1
- net GND1: now also C4.2, C3.2, U5.7 (nOUT1)
- net GND2: now also C43.2, C42.2, C62.1, U5.9 (GND_2); no longer X1.9
- net IN_WH: now also C62.2
- net H+15V: no longer names the net of X1.10
Other:
- moved on the sheet: C48, R53

Commit message: change IPM to STGIF7CH60TS
Parts:
- removed BC2, C39, C4, C40, C41, C43, C47, C50, C51, C54, C60, C61: 104, Capacitor_SMD:C_0805_2012Metric_Pad1.18x1.45mm_HandSolder, symbol Device:C
- removed BX1, BX2, BX3, BX4: BLM31KN801SH1L, Resistor_SMD:R_1206_3216Metric_Pad1.30x1.75mm_HandSolder, symbol bead:bead
- removed C10, C11, C16, C17, C18, C19, C20, C23, C26, C32, C33, C34, C36, C6, C7, C9: 104, Capacitor_SMD:C_0805_2012Metric, symbol Device:C
- removed C2, C3, C42, C45, C46, C48, C49: 470uF/25V, Capacitor_SMD:CP_Elec_10x12.5, symbol Device:C_Polarized
- removed C22: 470uF/400V, inv24VLib:CAPPRD1000W160D3600H5200, symbol Device:C_Polarized
- removed C35: 2200uF/50V, Capacitor_THT:CP_Radial_D12.5mm_P7.50mm, symbol Device:C_Polarized
- removed C52, C55: 220uF/50V, Capacitor_SMD:CP_Elec_10x12.5, symbol Device:C_Polarized
- removed C53: 334, Capacitor_SMD:C_0805_2012Metric_Pad1.18x1.45mm_HandSolder, symbol Device:C
- removed D8: BYV29X-500, inv24VLib:TO507P1020X460X2000-2, symbol bead:D_Schottky
- removed R59: 22, Resistor_SMD:R_2010_5025Metric_Pad1.40x2.65mm_HandSolder, symbol Device:R
- removed RV4: ERZ-VF2M560, inv24VLib:VAR_ERZ-VF2M560, symbol ERZ-VF2M560:ERZ-VF2M560
- removed X1: ~, inv24VLib:ee42208x8p, symbol bead:EE4220_8x8P
- added BC10, BC11, BC12, BC13, BC14, BC15, BC16, BC17, BC18, BC19, BC2, BC20, BC21, BC22, BC23, BC24, BC25, BC26, BC27, BC28, BC29, BC3, BC30, BC31, BC4, BC5, BC6, BC7, BC8, BC9: 104/50V, mod:CAPC2012X95N, symbol CL21B104KBCNNND:CL21B104KBCNNND
- added BX1, BX2, BX3, BX4: 2.5A/0.8K, mod:BLM31KN102BH1L, symbol BLM31KN801SH1L:BLM31KN801SH1L
- added C2, C3, C45, C48, C52, C55, C6: 680uF/25V, Capacitor_SMD:CP_Elec_16x17.5, symbol MAL226099105E3:MAL226099105E3
- added C22: 470uF/400V, Capacitor_THT:CP_Radial_D35.0mm_P10.00mm_SnapIn, symbol MAL226099105E3:MAL226099105E3
- added C4: 2200uF/50V, Capacitor_THT:CP_Radial_D18.0mm_P7.50mm, symbol Device:C_Polarized
- added D8: BYV29X-600, mod:TO507P1020X460X2000-2, symbol Diode:1N5822
- added L6: L_Ferrite_Coupled_1423, Inductor_THT:L_CommonMode_Toroid_Vertical_L39.4mm_W20.3mm_Px15.24mm_Py22.86mm_Bourns_8100, symbol Device:L_Ferrite_Coupled_1423
- added Q7: SUP53P06-20-E3, mod:TO254P465X1028X1931-3P, symbol SUP53P06-20-E3:SUP53P06-20-E3
- added R50: 1K, Resistor_SMD:R_0805_2012Metric_Pad1.20x1.40mm_HandSolder, symbol Device:R
- added RT1: MS35_1R040, mod:MS351R040, symbol MS35_1R040:MS35_1R040
- added TR1: pq5050v, mod:pq5050h, symbol pq5050:pq5050v
- added Z1: SZMMSZ4699T1G, mod:SOD3716X135N, symbol SZMMSZ4699T1G:SZMMSZ4699T1G
- BC1: value 104 -> 104/50V; footprint Capacitor_SMD:C_0805_2012Metric_Pad1.18x1.45mm_HandSolder -> mod:CAPC2012X95N; symbol Device:C -> CL21B104KBCNNND:CL21B104KBCNNND; Height (none) -> 0.95; Manufacturer_Name (none) -> SAMSUNG; Manufacturer_Part_Number (none) -> CL21B104KBCNNNE; Mouser Part Number (none) -> 187-CL21B104KBCNNNE; Mouser Price/Stock (none) -> https://www.mouser.co.uk/ProductDetail/Samsung-Electro-Mech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
- C1: footprint Capacitor_THT:CP_Radial_D12.5mm_P7.50mm -> Capacitor_THT:CP_Radial_D18.0mm_P7.50mm; Manufacturer_Name (none) -> Samyoung; Manufacturer_Part_Number (none) -> NXA 50V 2200uF
- C12, C25, C27, C28, C30, C31, C5, C62, C8: Cost (none) -> 20; Manufacturer_Name (none) -> SAMSUNG; Manufacturer_Part_Number (none) -> CL21B102KBCNNNE; Mouser Part Number (none) -> 187-CL21B104KBCNNNE; Mouser Price/Stock (none) -> https://www.mouser.co.uk/ProductDetail/Samsung-Electro-Mech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
- C13, C14, C15: footprint Capacitor_SMD:C_0805_2012Metric -> Capacitor_SMD:C_1210_3225Metric_Pad1.33x2.70mm_HandSolder; Cost (none) -> 402; Manufacturer_Name (none) -> SAMSUNG; Manufacturer_Part_Number (none) -> CL32B226KAJNNNE; Mouser Part Number (none) -> 187-CL32B226KAJNNNE; Mouser Price/Stock (none) -> https://www.mouser.kr/ProductDetail/Samsung-Electro-Mechani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
- C21: value 104 -> 102
- C24: Cost (none) -> 20; Manufacturer_Name (none) -> SAMSUNG; Manufacturer_Part_Number (none) -> CL21B333KBCNNNE; Mouser Part Number (none) -> 187-CL21B333KBCNNNE; Mouser Price/Stock (none) -> https://www.mouser.co.uk/ProductDetail/Samsung-Electro-Mech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
- C37, C38: footprint Capacitor_SMD:C_0805_2012Metric_Pad1.18x1.45mm_HandSolder -> Capacitor_SMD:C_0805_2012Metric; Cost (none) -> 20; Manufacturer_Name (none) -> SAMSUNG; Manufacturer_Part_Number (none) -> CL21B103KBCNNNE; Mouser Part Number (none) -> 187-CL21B103KBCNNNE; Mouser Price/Stock (none) -> https://www.mouser.co.uk/ProductDetail/Samsung-Electro-Mech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
- C56: footprint Resistor_THT:R_Axial_DIN0207_L6.3mm_D2.5mm_P10.16mm_Horizontal -> Capacitor_SMD:C_1812_4532Metric_Pad1.57x3.40mm_HandSolder; Cost (none) -> 917; Manufacturer_Name (none) -> Vishay / Vitramon; Manufacturer_Part_Number (none) -> VJ1808Y103KXGAT; Mouser Part Number (none) -> 77-VJ1808Y103KXGAT; Mouser Price/Stock (none) -> https://www.mouser.kr/ProductDetail/Vishay-Vitramon/VJ1808Y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
- D1, D2, D6, D7: value SS16 -> SS26; footprint Diode_SMD:D_3220_8050Metric_Pad2.65x5.15mm_HandSolder -> mod:DIOM5127X229N; Cost (none) -> 500; Height (none) -> 2.29; Manufacturer_Name (none) -> Vishay; Manufacturer_Part_Number (none) -> SS26SHE3_B/H; Mouser Part Number (none) -> 78-SS26SHE3_B/H; Mouser Price/Stock (none) -> https://www.mouser.co.uk/ProductDetail/Vishay-General-Semic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
- D3, D4, D5: value ES1F-ES1J -> ES1F; footprint Diode_SMD:D_2114_3652Metric_Pad1.85x3.75mm_HandSolder -> mod:DIOM5027X244N; Cost (none) -> 500; Height (none) -> 2.29; Manufacturer_Name (none) -> onsemi / Fairchild; Manufacturer_Part_Number (none) -> ES1F; Mouser Part Number (none) -> 512-ES1F; Mouser Price/Stock (none) -> https://www.mouser.kr/ProductDetail/onsemi-Fairchild/ES1F?q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
- SW1: footprint inv24VLib:PDIP4GW_709AH_ONS-M -> mod:418117270902; symbol Switch:SW_DIP_x02 -> 418117270902:418117270902; Availability (none) -> In Stock; Check_prices (none) -> https://www.snapeda.com/parts/418117270902/Wurth+Elektronik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; DATASHEET-URL (none) -> https://www.we-online.com/catalog/datasheet/418117270902.pdf; Description_1 (none) -> Dip Switch SPST 2 Position Through Hole Slide (Standard) Ac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; MF (none) -> Würth Elektronik; MP (none) -> 418117270902; PART-NUMBER (none) -> 418117270902; PINS (none) -> 2; Package (none) -> None; Price (none) -> None; QTY (none) -> 82; SnapEDA_Link (none) -> https://www.snapeda.com/parts/418117270902/Wurth+Elektronik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
Connections:
- net +15V: now also BC14.1
- net +24V: now also D9.1 (K), U2.5 (ON/OFF), BC26.1, C4.1, Q7.3 (S), TR1.4, TR1.5, Z1.1 (K); no longer F1.2_1, F1.2_2, RV1.2, RV2.2, RV3.2, U2.1 (VIN)
- net +3.3V: now also BC15.1, BC7.1
- net +5P: now also BC1.1, C38.1, BC2.1, BC27.1, C55.1 (+); no longer BC1.2, C38.2
- net +5V: now also BC16.1, BC19.1, BC4.2, BC5.1, BX1.1, C2.1 (+)
- net +5VP: now also BC13.1, BC25.1, BC6.1, BC8.1, C48.1 (+)
- net +8VP_IN: now also BC3.1, C3.1 (+)
- net +BATT: now also BC31.1, C52.1 (+)
- net 15V_H_IN: now also BC23.1, C6.1 (+)
- net DIN_A: now also SW1.2, BC29.1; no longer SW1.4
- net DIN_B: now also SW1.1, BC30.1; no longer SW1.3
- net Earth: now also C56.1, RV2.2, RV3.2; no longer C56.2
- net GND: now also C37.2, C56.2, SW1.A1, SW1.A2, U2.1 (VIN), BC12.2, BC15.2, BC16.2, BC18.2, BC19.2, BC26.2, BC29.2, BC30.2, BC4.1, BC5.2, BC7.2, BX2.1, C2.2 (-), C4.2, L6.3, R50.1; no longer C37.1, C56.1, D9.2 (A), F2.2_1, F2.2_2, RV1.1, SW1.1, SW1.2, U2.5 (ON/OFF)
- net GND1: now also BC1.2, C38.2, BC2.2, BC20.2, BC21.2, BC22.2, BC27.2, BC3.2, BC31.2, C3.2 (-), C52.2 (-), C55.2 (-); no longer BC1.1, C38.1
- net GND2: now also C12.2, C27.2, C28.2, C30.2, C31.2, C62.2, BC13.2, BC14.2, BC23.2, BC24.2, BC25.2, BC6.2, BC8.2, BX3.1, C45.2 (-), C48.2 (-), C6.2 (-); no longer C12.1, C27.1, C28.1, C30.1, C31.1, C62.1
- net GNDPWR: now also BX3.2, C22.2 (-), TR1.12, TR1.13
- net IN_UH: now also C27.1; no longer C27.2
- net IN_UL: now also C12.1; no longer C12.2
- net IN_VH: now also C28.1; no longer C28.2
- net IN_VL: now also C30.1; no longer C30.2
- net IN_WH: now also C62.1; no longer C62.2
- net IN_WL: now also C31.1; no longer C31.2
- net RX_CAN: now also C37.1; no longer C37.2
- net TEMPERATURE_IPM: now also BC18.1, BX4.1
- net VBUS: now also C22.1 (+)
- net VDC_IN: now also BC12.1
- net VTH_IPM: now also BC17.1, BX1.2
- net at C15.1, D5.1 (K), IC1.13 (VB(U)): now also BC11.1
- net at C15.2, IC1.14 (VS(U)), R13.2: now also BC11.2
- net at L3.2, TP2.1, U12.1 (VIN): now also BC24.1, C45.1 (+)
- net at C13.2, IC1.23 (VS(W)), R11.2: now also BC9.2
- net at J1.4, R49.2, U11.3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: now also BC21.1
- net at J1.3, R48.2, U11.4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: now also BC22.1
- net at RV3.1: now also F1.2_1, F1.2_2, RV1.1, RT1.1; no longer RV2.1
- net at C14.2, IC1.19 (VS(V)), R12.2: now also BC10.2
- net at C14.1, D3.1 (K), IC1.18 (VB(V)): now also BC10.1
- net at R47.1, R48.1, R49.1: now also BC20.1
- net at L4.2: now also D8.1 (K)
- net at C13.1, D4.1 (K), IC1.22 (VB(W)): now also BC9.1
- net at IC1.25 (RTH): now also BX4.2
- net at Q2.2 (D): now also TR1.8
- net at Q1.2 (D): now also TR1.1
- net at F2.1_2, J10.1 (Pin_1): no longer F2.1_1
- new net: D9.2 (A), L6.4, Q7.2 (D)
- new net: BC28.2, F2.2_1, F2.2_2, L6.2, RV1.2, RV2.1
- new net: BC28.1, L6.1, RT1.2
- new net: Q7.1 (G), R50.2, Z1.2 (A)
- new net: BC17.2, BX2.2
- new net 300V_OUT1: TR1.16
- new net 300V_OUT2: D8.2 (A), TR1.9
Other:
- moved on the sheet: C1, C29, F1, F2, L1, L4, Q1, Q3, Q5, R1, R3, R5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
